File: hardware/HixCO2TemperatureIRBlaster.sch (EAGLE design)
At the start: 38 parts, among them J1 FTDI, J2 IEC320C8, J3 XH4P, Q1 AO3400, Q2 AO3400, U1 TSOP2238, U2 LM3940, U3 HLK-PM01, U4 DS18B20

Commit message: Fixed short-circuit between 3.3V and 5.0V on board layout
Changed lines of the file:
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@@
 <part name="GND5" library="supply1" library_urn="urn:adsk.eagle:library:371" deviceset="GND" device=""/>
 <part name="SUPPLY4" library="0_HixField" library_urn="urn:adsk.eagle:library:13392178" deviceset="3.3V" device=""/>
-<part name="U1" library="0_HixField" library_urn="urn:adsk.eagle:library:13392178" deviceset="TSOP2238" device="" package3d_urn="urn:adsk.eagle:package:17848656/4" value="TSOP2238"/>
+<part name="U1" library="0_HixField" library_urn="urn:adsk.eagle:library:13392178" deviceset="TSOP2238" device="" package3d_urn="urn:adsk.eagle:package:17848656/5" value="TSOP2238"/>
 <part name="U$3" library="0_HixField" library_urn="urn:adsk.eagle:library:13392178" deviceset="LED_RGB" device="" package3d_urn="urn:adsk.eagle:package:17854569/4"/>
 <part name="GND9" library="supply1" deviceset="GND" device=""/>
@@
 </instance>
 <instance part="FRAME1" gate="G$1" x="-10.16" y="-45.72" smashed="yes">
-<attribute name="DRAWING_NAME" x="207.01" y="-30.48" size="2.54" layer="94"/>
+<attribute name="DRAWING_NAME" x="207.01" y="-30.48" size="1.905" layer="94"/>
 <attribute name="LAST_DATE_TIME" x="207.01" y="-35.56" size="2.286" layer="94"/>
 <attribute name="SHEET" x="220.345" y="-40.64" size="2.54" layer="94"/>
